File: PicoMicrocontroller.kicad_sch (KiCad schematic)
At the start: 25 parts, among them J8 RUN, Q1 Q_PMOS_GSD, U6 Pico

Commit message: Finished schematic. Move to PCB.
Parts:
- removed C1: 1uF, Capacitor_SMD:C_0805_2012Metric, symbol Device:C
- removed D49: D, Diode_SMD:D_SOD-123, symbol Device:D
- removed Q1: Q_PMOS_GSD, Package_TO_SOT_SMD:SOT-23, symbol Device:Q_PMOS_GSD
- removed R63: NSΩ, Resistor_SMD:R_0805_2012Metric, symbol Device:R
- added C10, C15: 10uF, Capacitor_SMD:C_0805_2012Metric, symbol Device:C
- added C11, C23, C31, C8, C9: 1uF, Capacitor_SMD:C_0805_2012Metric, symbol Device:C
- added R63 (x3): 100kΩ, Resistor_SMD:R_0805_2012Metric, symbol Device:R
- added U1, U2, U5: MAX40200AUK, Package_TO_SOT_SMD:SOT-23-5, symbol Analog_Switch:MAX40200AUK
- J8: footprint (none) -> Connector_PinHeader_2.54mm:PinHeader_1x02_P2.54mm_Vertical
- renumbered C15 to C32, C15 to C5, FB8 to FB1
Connections:
- net +3.3V: now also C10.1, U5.5 (OUT)
- net +5V: now also C15.1, C8.1, R63.2, U2.1 (VDD); no longer C32.1
- net GND: now also C10.2, C11.2, C15.2, C23.2, C31.2, C8.2, C9.2, U1.2 (GND), U2.2 (GND), U5.2 (GND)
- net at U6.40 (VBUS): now also R63.2, U1.1 (VDD)
- net at R63.2, U6.39 (VSYS): now also C32.1, C9.1, U1.5 (OUT), U2.5 (OUT)
- net at C5.1, U6.36 (3V3): now also R63.2, U5.1 (VDD)
- new net: C11.1, R63.1, U5.3 (EN)
- new net: C23.1, R63.1, U1.3 (EN)
- new net: C31.1, R63.1, U2.3 (EN)
Other:
- moved on the sheet: C32, C5, D39, FB1, J8, R26, R63, U6
