File: PicoIrrigation.kicad_sch (KiCad schematic)
At the start: 4 parts, among them J1 M3, J2 M3, J3 M3, J4 M3

Commit message: Finished layout
Changed lines of the file:
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@@
     (effects (font (size 1.27 1.27)) (justify left bottom))
   )
-  (label "CS0" (at 65.024 96.266 0) (fields_autoplaced)
+  (label "CS1" (at 65.024 96.266 0) (fields_autoplaced)
     (effects (font (size 1.27 1.27)) (justify left bottom))
   )
@@
     (effects (font (size 1.27 1.27)) (justify left bottom))
   )
-  (label "CS0" (at 71.12 165.862 180) (fields_autoplaced)
+  (label "CS1" (at 71.12 165.862 180) (fields_autoplaced)
     (effects (font (size 1.27 1.27)) (justify right bottom))
   )
@@
       (effects (font (size 1.27 1.27)) (justify right))
     )
-    (pin "CS1" input (at 57.404 77.216 0)
+    (pin "CS1" input (at 57.404 96.266 0)
       (effects (font (size 1.27 1.27)) (justify right))
     )
@@
       (effects (font (size 1.27 1.27)) (justify right))
     )
-    (pin "CS0" input (at 57.404 96.266 0)
-      (effects (font (size 1.27 1.27)) (justify right))
-    )
+    (pin "CS0" input (at 57.404 77.216 0)
+      (effects (font (size 1.27 1.27)) (justify right))
+    )
